Commit message: missing transmission now simulation works

File: robots/jumpleg.urdf.xacro (robot description, xacro)
@@ -7,4 +7,39 @@
         <xacro:arg name="task_period" value="$(arg task_period)"/>
     </xacro:include>
+    <xacro:include filename="$(find jumpleg_description)/urdfs/floatingbase.transmission.xacro"/>
+	 <link name="world"/>
+ 	<joint name="base_x_joint" type="prismatic">
+		<parent link="world"/>
+		<child link="fake_link1"/>
+		<axis xyz="1 0 0 "/>
+		<origin xyz="0 0 0" rpy="0 0 0"/>
+		<limit effort="150" velocity="100.0" lower="-100" upper="100"/>
+	</joint>
+	<link name="fake_link1">
+	<inertial>
+	<mass value="0.00001"/>
+	<inertia ixx="5.8083e-4" ixy="0" ixz="0" iyy="3.0833e-5" iyz="0" izz="5.9083e-4"/>
+	</inertial>
+	</link>
+	<joint name="base_y_joint" type="prismatic">
+		<parent link="fake_link1"/>
+		<child link="fake_link2"/>
+		<axis xyz="0 1 0 "/>
+		<origin xyz="0 0 0" rpy="0 0 0"/>
+		<limit effort="150" velocity="100.0" lower="-100" upper="100"/>
+	</joint>
+	<link name="fake_link2">
+	<inertial>
+	<mass value="0.00001"/>
+	<inertia ixx="5.8083e-4" ixy="0" ixz="0" iyy="3.0833e-5" iyz="0" izz="5.9083e-4"/>
+	</inertial>
+	</link>
+	<joint name="base_z_joint" type="prismatic">
+		<parent link="fake_link2"/>
+		<child link="base_link"/>
+		<axis xyz="0 0 1 "/>
+		<origin xyz="0 0 0" rpy="0 0 0"/>
+		<limit effort="150" velocity="100.0" lower="-100" upper="100"/>
+	</joint>
       <link name="base_link"/>
     <joint name="floating_base" type="fixed">
@@ -25,5 +60,5 @@
             <origin xyz="0 0 0" rpy="0 0 0" />
             <geometry>
-          	 <box size="0.25 0.25 0.25"/>
+          	 <box size="0.05 0.05 0.05"/>
             </geometry>
                 <material name="${color_name}">
@@ -34,5 +69,5 @@
             <origin xyz="0 0 0" rpy="0 0 0" />
             <geometry>
-		 <box size="0.25 0.25 0.25"/>
+		 <box size="0.05 0.05 0.05"/>
 	   </geometry>
             <material name="${color_name}">
@@ -57,3 +92,4 @@
 	    color="${color}"
 	    opacity="${opacity}"/>
+         <xacro:floating_base_transmission name=""/>
 </robot>
