Commit message: now torque and kin limits are parametric!

File: urdf/jumpleg.xacro (robot description, xacro)
@@ -14,5 +14,5 @@
 		<axis xyz="1 0 0 "/>
 		<origin xyz="0 0 0" rpy="0 0 0"/>
-		<limit effort="150" velocity="100.0" lower="-100" upper="100"/>
+		<limit effort="1000" velocity="100.0" lower="-100" upper="100"/>
 	</joint>
 	<link name="fake_link1">
@@ -27,5 +27,5 @@
 		<axis xyz="0 1 0 "/>
 		<origin xyz="0 0 0" rpy="0 0 0"/>
-		<limit effort="150" velocity="100.0" lower="-100" upper="100"/>
+		<limit effort="1000" velocity="100.0" lower="-100" upper="100"/>
 	</joint>
 	<link name="fake_link2">
@@ -40,5 +40,5 @@
 		<axis xyz="0 0 1 "/>
 		<origin xyz="0 0 0" rpy="0 0 0"/>
-		<limit effort="150" velocity="100.0" lower="-100" upper="100"/>
+		<limit effort="1000" velocity="100.0" lower="-100" upper="100"/>
 	</joint>
       <link name="base_link"/>

File: urdf/leg.xacro (robot description, xacro)
@@ -4,4 +4,5 @@
     <xacro:include filename="$(find jumpleg_description)/urdf/leg.transmission.xacro"/>
     <xacro:include filename="$(find jumpleg_description)/urdf/leg.gazebo.xacro"/>
+    <xacro:include filename="$(find jumpleg_description)/urdf/commons.xacro"/>
     <!-- These are absoulte distance value, the sign are decided below -->
     <xacro:property name="base_2_HAA_x" value="0" />
@@ -14,9 +15,7 @@
     <xacro:property name="KFE_2_FOOT_y" value="${8.0 * 0.001}" />
     <xacro:property name="KFE_2_FOOT_z" value="${160.00 * 0.001}" />
-    <xacro:property name="MAX_TORQUE" value="1.2" />
     <!-- This macro has for purpose to define a leg -->
     <xacro:macro name="leg" params="prefix is_front is_right has_side_motion
                                   color_name color opacity">
-        <!-- Solo12 -->
         <xacro:if value="${has_side_motion}">
             <!--HAA JOINT: Joint between the trunk and the hip assembly -->
@@ -31,5 +30,5 @@
                         <!-- LF_HAA_JOINT -->
                         <!-- lower=-75deg, upper=140, velocity=555.5rpm (=5000rpm motor-side) -->
-                        <limit effort="${MAX_TORQUE}" lower="-1.30899694" upper="2.44346095" velocity="58.17764173"/>
+                        <limit effort="${MAX_TORQUE}" lower="${haa_min}" upper="${haa_max}" velocity="58.17764173"/>
                         <origin xyz="${base_2_HAA_x} ${base_2_HAA_y} 0" rpy="0 0 0" />
                     </xacro:unless>
@@ -37,5 +36,5 @@
                         <!-- RF_HAA_JOINT -->
                         <!-- lower=-140deg, upper=75, velocity=555.5rpm (=5000rpm motor-side) -->
-                        <limit effort="${MAX_TORQUE}" lower="-2.44346095" upper="1.30899694" velocity="58.17764173"/>
+                        <limit effort="${MAX_TORQUE}" lower="-${haa_max}" upper="-${haa_min}" velocity="58.17764173"/>
                         <origin xyz="${base_2_HAA_x} ${-base_2_HAA_y} 0" rpy="0 0 0" />
                     </xacro:if>
@@ -45,5 +44,5 @@
                         <!-- LH_HAA_JOINT -->
                         <!-- lower=-75deg, upper=140, velocity=555.5rpm (=5000rpm motor-side) -->
-                        <limit effort="${MAX_TORQUE}" lower="-1.30899694" upper="2.44346095" velocity="58.17764173"/>
+                        <limit effort="${MAX_TORQUE}" lower="${haa_min}" upper="${haa_max}" velocity="58.17764173"/>
                         <origin xyz="${-base_2_HAA_x} ${base_2_HAA_y} 0" rpy="0 0 0" />
                     </xacro:unless>
@@ -51,5 +50,5 @@
                         <!-- RH_HAA_JOINT -->
                         <!-- lower=-140deg, upper=75, velocity=555.5rpm (=5000rpm motor-side) -->
-                        <limit effort="${MAX_TORQUE}" lower="-2.44346095" upper="1.30899694" velocity="58.17764173"/>
+                        <limit effort="${MAX_TORQUE}" lower="-${haa_max}" upper="-${haa_min}" velocity="58.17764173"/>
                         <origin xyz="${-base_2_HAA_x} ${-base_2_HAA_y} 0" rpy="0 0 0" />
                     </xacro:if>
@@ -185,5 +184,5 @@
                         <!-- LF_HFE_JOINT -->
                         <!-- lower=-225deg, upper=90deg, velocity=555.5rpm (=5000rpm motor-side) -->
-                        <limit effort="${MAX_TORQUE}" lower="-3.92699082" upper="1.57079633" velocity="58.17764173"/>
+                        <limit effort="${MAX_TORQUE}" lower="${hfe_min}" upper="${hfe_max}" velocity="58.17764173"/>
                         <origin xyz="0 ${HAA_2_HFE_y} 0" rpy="0 0 0" />
                     </xacro:unless>
@@ -191,5 +190,5 @@
                         <!-- RF_HFE_JOINT -->
                         <!-- lower=-225deg, upper=90deg, velocity=555.5rpm (=5000rpm motor-side) -->
-                        <limit effort="${MAX_TORQUE}" lower="-3.92699082" upper="1.57079633" velocity="58.17764173"/>
+                        <limit effort="${MAX_TORQUE}" lower="${hfe_min}" upper="${hfe_max}" velocity="58.17764173"/>
                         <origin xyz="0 ${-HAA_2_HFE_y} 0" rpy="0 0 0" />
                     </xacro:if>
@@ -199,5 +198,5 @@
                         <!-- LH_HFE_JOINT -->
                         <!-- lower=-90deg, upper=225deg, velocity=555.5rpm (=5000rpm motor-side) -->
-                        <limit effort="${MAX_TORQUE}" lower="-1.57079633" upper="3.92699082" velocity="58.17764173"/>
+                        <limit effort="${MAX_TORQUE}" lower="-${hfe_max}" upper="-${hfe_min}" velocity="58.17764173"/>
                         <origin xyz="0 ${HAA_2_HFE_y} 0" rpy="0 0 0" />
                     </xacro:unless>
@@ -205,5 +204,5 @@
                         <!-- RF_HFE_JOINT -->
                         <!-- lower=-90deg, upper=225deg, velocity=555.5rpm (=5000rpm motor-side) -->
-                        <limit effort="${MAX_TORQUE}" lower="-1.57079633" upper="3.92699082" velocity="58.17764173"/>
+                        <limit effort="${MAX_TORQUE}" lower="-${hfe_max}" upper="-${hfe_min}" velocity="58.17764173"/>
                         <origin xyz="0 ${-HAA_2_HFE_y} 0" rpy="0 0 0" />
                     </xacro:if>
@@ -313,5 +312,5 @@
                     <!-- LF_KFE JOINT -->
                     <!-- lower=-370deg, upper=370deg, velocity=555.5rpm (=5000rpm motor-side) -->
-                    <limit effort="${MAX_TORQUE}" lower="-6.45771823" upper="6.45771823" velocity="58.17764173"/>
+                    <limit effort="${MAX_TORQUE}" lower="${kfe_min}" upper="${kfe_max}" velocity="58.17764173"/>
                     <origin xyz="0 ${HFE_2_KFE_y} ${-HFE_2_KFE_z}" rpy="0 0 0" />
                 </xacro:unless>
@@ -319,5 +318,5 @@
                     <!-- RF_KFE JOINT -->
                     <!-- lower=-370deg, upper=370deg, velocity=555.5rpm (=5000rpm motor-side) -->
-                    <limit effort="${MAX_TORQUE}" lower="-6.45771823" upper="6.45771823" velocity="58.17764173"/>
+                    <limit effort="${MAX_TORQUE}" lower="${kfe_min}" upper="${kfe_max}" velocity="58.17764173"/>
                     <origin xyz="0 ${-HFE_2_KFE_y} ${-HFE_2_KFE_z}" rpy="0 0 0" />
                 </xacro:if>
@@ -327,5 +326,5 @@
                     <!-- LH_KFE JOINT -->
                     <!-- lower=-370deg, upper=370deg, velocity=555.5rpm (=5000rpm motor-side) -->
-                    <limit effort="${MAX_TORQUE}" lower="-6.45771823" upper="6.45771823" velocity="58.17764173"/>
+                    <limit effort="${MAX_TORQUE}" lower="${kfe_min}" upper="${kfe_max}" velocity="58.17764173"/>
                     <origin xyz="0 ${HFE_2_KFE_y} ${-HFE_2_KFE_z}" rpy="0 0 0" />
                 </xacro:unless>
@@ -333,5 +332,5 @@
                     <!-- RH_KFE JOINT -->
                     <!-- lower=-370deg, upper=370deg, velocity=555.5rpm (=5000rpm motor-side) -->
-                    <limit effort="${MAX_TORQUE}" lower="-6.45771823" upper="6.45771823" velocity="58.17764173"/>
+                    <limit effort="${MAX_TORQUE}" lower="${kfe_min}" upper="${kfe_max}" velocity="58.17764173"/>
                     <origin xyz="0 ${-HFE_2_KFE_y} ${-HFE_2_KFE_z}" rpy="0 0 0" />
                 </xacro:if>
