Commit message: adding common.xacro with torque and kin limits

File: urdf/common.xacro (robot description, xacro)
@@ -10,4 +10,4 @@
     <xacro:property name="kfe_min" value="-6.45771823"/>
     <!-- torque limits -->
-    <xacro:property name="MAX_TORQUE" value="1000" />
+    <xacro:property name="MAX_TORQUE" value="10" />
 </robot>

File: urdf/jumpleg.xacro (robot description, xacro)
@@ -8,4 +8,6 @@
     </xacro:include>
     <xacro:include filename="$(find jumpleg_description)/urdf/floatingbase.transmission.xacro"/>
+    <!-- The following included files set up definitions of parts of the robot body -->
+    <xacro:include filename="$(find jumpleg_description)/urdf/common.xacro"/>
 	 <link name="world"/>
  	<joint name="base_x_joint" type="prismatic">

Commit message: reduced soft limits to avoid leg being stuck

File: urdf/common.xacro (robot description, xacro)
@@ -9,4 +9,8 @@
     <xacro:property name="kfe_max" value="6.45771823"/>
     <xacro:property name="kfe_min" value="-6.45771823"/>
+    <xacro:property name="haa_max_soft" value="2.43"/>
+    <xacro:property name="haa_min_soft" value="-1.25"/>
+    <xacro:property name="hfe_max_soft" value="1.53"/>
+    <xacro:property name="hfe_min_soft" value="-3.8"/>
     <!-- torque limits -->
     <xacro:property name="MAX_TORQUE" value="10" />

File: urdf/leg.xacro (robot description, xacro)
@@ -30,5 +30,5 @@
                         <!-- lower=-75deg, upper=140, velocity=555.5rpm (=5000rpm motor-side) -->
                         <limit effort="${MAX_TORQUE}" lower="${haa_min}" upper="${haa_max}" velocity="58.17764173"/>
-			<safety_controller k_position="10" k_velocity="1"   soft_lower_limit="${haa_min}" soft_upper_limit="${haa_max}" />
+			<safety_controller k_position="10" k_velocity="1"   soft_lower_limit="${haa_min_soft}" soft_upper_limit="${haa_max_soft}" />
                         <origin xyz="${base_2_HAA_x} ${base_2_HAA_y} 0" rpy="0 0 0" />
                     </xacro:unless>
@@ -37,5 +37,5 @@
                         <!-- lower=-140deg, upper=75, velocity=555.5rpm (=5000rpm motor-side) -->
                         <limit effort="${MAX_TORQUE}" lower="-${haa_max}" upper="-${haa_min}" velocity="58.17764173"/>
-			<safety_controller k_position="10" k_velocity="1"   soft_lower_limit="-${haa_max}" soft_upper_limit="-${haa_min}" />
+			<safety_controller k_position="10" k_velocity="1"   soft_lower_limit="-${haa_max_soft}" soft_upper_limit="-${haa_min_soft}" />
                         <origin xyz="${base_2_HAA_x} ${-base_2_HAA_y} 0" rpy="0 0 0" />
                     </xacro:if>
@@ -46,5 +46,5 @@
                         <!-- lower=-75deg, upper=140, velocity=555.5rpm (=5000rpm motor-side) -->
                         <limit effort="${MAX_TORQUE}" lower="${haa_min}" upper="${haa_max}" velocity="58.17764173"/>
-			<safety_controller k_position="10" k_velocity="1"   soft_lower_limit="${haa_min}" soft_upper_limit="${haa_max}" />
+			<safety_controller k_position="10" k_velocity="1"   soft_lower_limit="${haa_min_soft}" soft_upper_limit="${haa_max_soft}" />
                         <origin xyz="${-base_2_HAA_x} ${base_2_HAA_y} 0" rpy="0 0 0" />
                     </xacro:unless>
@@ -53,5 +53,5 @@
                         <!-- lower=-140deg, upper=75, velocity=555.5rpm (=5000rpm motor-side) -->
                         <limit effort="${MAX_TORQUE}" lower="-${haa_max}" upper="-${haa_min}" velocity="58.17764173"/>
-			<safety_controller k_position="10" k_velocity="1"   soft_lower_limit="-${haa_max}" soft_upper_limit="-${haa_min}" />
+			<safety_controller k_position="10" k_velocity="1"   soft_lower_limit="-${haa_max_soft}" soft_upper_limit="-${haa_min_soft}" />
                         <origin xyz="${-base_2_HAA_x} ${-base_2_HAA_y} 0" rpy="0 0 0" />
                     </xacro:if>
@@ -188,5 +188,5 @@
                         <!-- lower=-225deg, upper=90deg, velocity=555.5rpm (=5000rpm motor-side) -->
                         <limit effort="${MAX_TORQUE}" lower="${hfe_min}" upper="${hfe_max}" velocity="58.17764173"/>
-			<safety_controller k_position="10" k_velocity="1"   soft_lower_limit="${hfe_min}" soft_upper_limit="${hfe_max}" />
+			<safety_controller k_position="10" k_velocity="1"   soft_lower_limit="${hfe_min_soft}" soft_upper_limit="${hfe_max_soft}" />
                         <origin xyz="0 ${HAA_2_HFE_y} 0" rpy="0 0 0" />
                     </xacro:unless>
@@ -195,5 +195,5 @@
                         <!-- lower=-225deg, upper=90deg, velocity=555.5rpm (=5000rpm motor-side) -->
                         <limit effort="${MAX_TORQUE}" lower="${hfe_min}" upper="${hfe_max}" velocity="58.17764173"/>
-			<safety_controller k_position="10" k_velocity="1"   soft_lower_limit="${hfe_min}" soft_upper_limit="${hfe_max}" />
+			<safety_controller k_position="10" k_velocity="1"   soft_lower_limit="${hfe_min_soft}" soft_upper_limit="${hfe_max_soft}" />
                         <origin xyz="0 ${-HAA_2_HFE_y} 0" rpy="0 0 0" />
                     </xacro:if>
@@ -204,5 +204,5 @@
                         <!-- lower=-90deg, upper=225deg, velocity=555.5rpm (=5000rpm motor-side) -->
                         <limit effort="${MAX_TORQUE}" lower="-${hfe_max}" upper="-${hfe_min}" velocity="58.17764173"/>
-			<safety_controller k_position="10" k_velocity="1"   soft_lower_limit="-${hfe_max}" soft_upper_limit="-${hfe_min}" />
+			<safety_controller k_position="10" k_velocity="1"   soft_lower_limit="-${hfe_max_soft}" soft_upper_limit="-${hfe_min_soft}" />
                         <origin xyz="0 ${HAA_2_HFE_y} 0" rpy="0 0 0" />
                     </xacro:unless>
@@ -211,5 +211,5 @@
                         <!-- lower=-90deg, upper=225deg, velocity=555.5rpm (=5000rpm motor-side) -->
                         <limit effort="${MAX_TORQUE}" lower="-${hfe_max}" upper="-${hfe_min}" velocity="58.17764173"/>
-			<safety_controller k_position="10" k_velocity="1"   soft_lower_limit="-${hfe_max}" soft_upper_limit="-${hfe_min}" />
+			<safety_controller k_position="10" k_velocity="1"   soft_lower_limit="-${hfe_max_soft}" soft_upper_limit="-${hfe_min_soft}" />
                         <origin xyz="0 ${-HAA_2_HFE_y} 0" rpy="0 0 0" />
                     </xacro:if>

Commit message: restroring torques to 10 Nm

File: urdf/common.xacro (robot description, xacro)
@@ -14,4 +14,4 @@
     <xacro:property name="hfe_min_soft" value="-1.45"/>
     <!-- torque limits real should be 1.57-->
-    <xacro:property name="MAX_TORQUE" value="2." />
+    <xacro:property name="MAX_TORQUE" value="10." />
 </robot>

Commit message: added crocoddyl urdf

File: urdf/common.xacro (robot description, xacro)
@@ -14,4 +14,4 @@
     <xacro:property name="hfe_min_soft" value="-1.45"/>
     <!-- torque limits real should be 1.57-->
-    <xacro:property name="MAX_TORQUE" value="10." />
+    <xacro:property name="MAX_TORQUE" value="5." />
 </robot>
